File: hardware/bmp/bmp.sch (KiCad schematic (older format))
At the start: 45 parts, among them J1 USB_C_Receptacle, J2 TC2050-IDC, J3 Conn_02x05_Odd_Even, J4 Conn_01x03, J5 Conn_01x04, Q1 SI2301CDS-T1-GE3, SW1 SW_Push, SW2 SW_Push, U1 XC6206P332MR, U2 STM32F103CBTx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

Commit message: updated with 2019 gdb
Parts:
- removed R6: 10k, Resistor_SMD:R_0603_1608Metric, symbol Device:R
- removed SW1: SW_Push, footprints:SW_TACT_TS-1145A_C318904, symbol Switch:SW_Push
- removed U1: XC6206P332MR, Package_TO_SOT_SMD:SOT-23, symbol Regulator_Linear:AP2127N-3.3
- added MH1, MH2: MountingHole, kbd:HOLE_JLCPCBA, symbol Mechanical:MountingHole
- added TP1: TestPoint_Probe, footprints:KB_BlueMicro, symbol Connector:TestPoint_Probe
- added U1: AP2112K-3.3, Package_TO_SOT_SMD:SOT-23-5, symbol E73:AP2112K-3.3
Connections:
- wire segments 224 -> 226
Changed lines of the file:
@@
 EESchema Schematic File Version 4
+LIBS:bmp-cache
 EELAYER 26 0
 EELAYER END
@@
 L power:+3.3V #PWR0102
 U 1 1 5EE0FD88
-P 2100 850
-F 0 "#PWR0102" H 2100 700 50  0001 C CNN
-F 1 "+3.3V" H 2115 1023 50  0000 C CNN
-F 2 "" H 2100 850 50  0001 C CNN
-F 3 "" H 2100 850 50  0001 C CNN
-	1    2100 850
+P 3000 850
+F 0 "#PWR0102" H 3000 700 50  0001 C CNN
+F 1 "+3.3V" H 3015 1023 50  0000 C CNN
+F 2 "" H 3000 850 50  0001 C CNN
+F 3 "" H 3000 850 50  0001 C CNN
+	1    3000 850
 	1    0    0    -1
 $EndComp
@@
 	900  1550 900  1650
 Wire Wire Line
-	900  1650 1350 1650
-Connection ~ 1350 1650
+	900  1650 1250 1650
 Wire Wire Line
 	1350 1650 1350 1750
@@
 L Device:C_Small C2
 U 1 1 5EE1D9D2
-P 2100 1300
-F 0 "C2" H 2192 1346 50  0000 L CNN
-F 1 "10uF" H 2192 1255 50  0000 L CNN
-F 2 "Capacitor_SMD:C_0603_1608Metric" H 2100 1300 50  0001 C CNN
-F 3 "~" H 2100 1300 50  0001 C CNN
-F 4 "C19702" H 2100 1300 50  0001 C CNN "LCSC"
-	1    2100 1300
-	1    0    0    -1
-$EndComp
-Wire Wire Line
-	2100 1400 2100 1650
-Wire Wire Line
-	2100 1650 1350 1650
-Wire Wire Line
-	1650 1150 2100 1150
-Wire Wire Line
-	2100 1150 2100 850
-Wire Wire Line
-	2100 1150 2100 1200
-Connection ~ 2100 1150
+P 3000 1300
+F 0 "C2" H 3092 1346 50  0000 L CNN
+F 1 "10uF" H 3092 1255 50  0000 L CNN
+F 2 "Capacitor_SMD:C_0603_1608Metric" H 3000 1300 50  0001 C CNN
+F 3 "~" H 3000 1300 50  0001 C CNN
+F 4 "C19702" H 3000 1300 50  0001 C CNN "LCSC"
+	1    3000 1300
+	1    0    0    -1
+$EndComp
+Wire Wire Line
+	3000 1400 3000 1650
+Wire Wire Line
+	2550 1150 3000 1150
+Wire Wire Line
+	3000 1150 3000 850
+Wire Wire Line
+	3000 1150 3000 1200
+Connection ~ 3000 1150
 Wire Wire Line
 	6050 4050 6250 4050
@@
 	-1   0    0    1
 $EndComp
-$Comp
-L Switch:SW_Push SW1
-U 1 1 5EE8D1E7
-P 4000 2700
-F 0 "SW1" H 4000 2985 50  0000 C CNN
-F 1 "SW_Push" H 4000 2894 50  0000 C CNN
-F 2 "footprints:SW_TACT_TS-1145A_C318904" H 4000 2900 50  0001 C CNN
-F 3 "" H 4000 2900 50  0001 C CNN
-F 4 "C318904" H 4000 2700 50  0001 C CNN "LCSC"
-	1    4000 2700
-	1    0    0    -1
-$EndComp
-$Comp
-L Device:R R6
-U 1 1 5EE8D39A
-P 3500 2700
-F 0 "R6" V 3293 2700 50  0000 C CNN
-F 1 "10k" V 3384 2700 50  0000 C CNN
-F 2 "Resistor_SMD:R_0603_1608Metric" V 3430 2700 50  0001 C CNN
-F 3 "~" H 3500 2700 50  0001 C CNN
-F 4 "C25804" V 3500 2700 50  0001 C CNN "LCSC"
-	1    3500 2700
-	0    1    1    0
-$EndComp
-$Comp
-L power:+3.3V #PWR0111
-U 1 1 5EE8D4AB
-P 4400 2500
-F 0 "#PWR0111" H 4400 2350 50  0001 C CNN
-F 1 "+3.3V" H 4415 2673 50  0000 C CNN
-F 2 "" H 4400 2500 50  0001 C CNN
-F 3 "" H 4400 2500 50  0001 C CNN
-	1    4400 2500
-	1    0    0    -1
-$EndComp
 Wire Wire Line
 	3350 3050 3350 2700
 Connection ~ 3350 3050
 Wire Wire Line
-	3650 2700 3750 2700
-Wire Wire Line
-	4200 2700 4400 2700
-Wire Wire Line
-	4400 2700 4400 2500
-Wire Wire Line
 	3750 2700 3750 2950
 Wire Wire Line
 	3750 2950 4750 2950
-Connection ~ 3750 2700
-Wire Wire Line
-	3750 2700 3800 2700
 Text Label 6250 4050 0    50   ~ 0
 iRST
@@
 L Device:C_Small C6
 U 1 1 5F1706E0
-P 2550 1300
-F 0 "C6" H 2642 1346 50  0000 L CNN
-F 1 "100nF" H 2642 1255 50  0000 L CNN
-F 2 "Capacitor_SMD:C_0603_1608Metric" H 2550 1300 50  0001 C CNN
-F 3 "~" H 2550 1300 50  0001 C CNN
-F 4 "C14663" H 2550 1300 50  0001 C CNN "LCSC"
-	1    2550 1300
+P 3450 1300
+F 0 "C6" H 3542 1346 50  0000 L CNN
+F 1 "100nF" H 3542 1255 50  0000 L CNN
+F 2 "Capacitor_SMD:C_0603_1608Metric" H 3450 1300 50  0001 C CNN
+F 3 "~" H 3450 1300 50  0001 C CNN
+F 4 "C14663" H 3450 1300 50  0001 C CNN "LCSC"
+	1    3450 1300
 	1    0    0    -1
 $EndComp
@@
 L Device:C_Small C7
 U 1 1 5F17077C
-P 2900 1300
-F 0 "C7" H 2992 1346 50  0000 L CNN
-F 1 "100nF" H 2992 1255 50  0000 L CNN
-F 2 "Capacitor_SMD:C_0603_1608Metric" H 2900 1300 50  0001 C CNN
-F 3 "~" H 2900 1300 50  0001 C CNN
-F 4 "C14663" H 2900 1300 50  0001 C CNN "LCSC"
-	1    2900 1300
-	1    0    0    -1
-$EndComp
-Wire Wire Line
-	2900 1200 2900 1150
-Wire Wire Line
-	2900 1150 2550 1150
-Wire Wire Line
-	2900 1400 2900 1650
-Wire Wire Line
-	2900 1650 2550 1650
-Connection ~ 2100 1650
-Wire Wire Line
-	2550 1400 2550 1650
-Connection ~ 2550 1650
-Wire Wire Line
-	2550 1650 2100 1650
-Wire Wire Line
-	2550 1200 2550 1150
-Connection ~ 2550 1150
-Wire Wire Line
-	2550 1150 2100 1150
+P 3800 1300
+F 0 "C7" H 3892 1346 50  0000 L CNN
+F 1 "100nF" H 3892 1255 50  0000 L CNN
+F 2 "Capacitor_SMD:C_0603_1608Metric" H 3800 1300 50  0001 C CNN
+F 3 "~" H 3800 1300 50  0001 C CNN
+F 4 "C14663" H 3800 1300 50  0001 C CNN "LCSC"
+	1    3800 1300
+	1    0    0    -1
+$EndComp
+Wire Wire Line
+	3800 1200 3800 1150
+Wire Wire Line
+	3800 1150 3450 1150
+Wire Wire Line
+	3800 1400 3800 1650
+Wire Wire Line
+	3800 1650 3450 1650
+Connection ~ 3000 1650
+Wire Wire Line
+	3450 1400 3450 1650
+Connection ~ 3450 1650
+Wire Wire Line
+	3450 1650 3000 1650
+Wire Wire Line
+	3450 1200 3450 1150
+Connection ~ 3450 1150
+Wire Wire Line
+	3450 1150 3000 1150
 $Comp
 L LOGIC-TXS0108EPWR_TSSOP20_:LOGIC-TXS0108EPWR(TSSOP20) U3
@@
 Connection ~ 8150 3350
 $Comp
-L Regulator_Linear:AP2127N-3.3 U1
-U 1 1 5F4D0A4A
-P 1350 1150
-F 0 "U1" H 1350 1392 50  0000 C CNN
-F 1 "XC6206P332MR" H 1350 1301 50  0000 C CNN
-F 2 "Package_TO_SOT_SMD:SOT-23" H 1350 1375 50  0001 C CIN
-F 3 "https://www.diodes.com/assets/Datasheets/AP2127.pdf" H 1350 1150 50  0001 C CNN
-F 4 "C5446" H 1350 1150 50  0001 C CNN "LCSC"
-	1    1350 1150
-	1    0    0    -1
-$EndComp
-Wire Wire Line
-	1050 1150 900  1150
-Wire Wire Line
-	1350 1450 1350 1650
+L E73:AP2112K-3.3 U1
+U 1 1 5EFA4751
+P 1950 850
+F 0 "U1" H 1925 887 60  0000 C CNN
+F 1 "AP2112K-3.3" H 1925 781 60  0000 C CNN
+F 2 "Package_TO_SOT_SMD:SOT-23-5" H 1950 150 60  0001 C CNN
+F 3 "" H 1950 150 60  0001 C CNN
+F 4 "C51118" H 1950 850 50  0001 C CNN "LCSC"
+	1    1950 850
+	1    0    0    -1
+$EndComp
+Wire Wire Line
+	900  1150 1100 1150
+Wire Wire Line
+	1300 1350 1100 1350
+Wire Wire Line
+	1100 1350 1100 1150
+Connection ~ 1100 1150
+Wire Wire Line
+	1100 1150 1300 1150
+Wire Wire Line
+	1300 1250 1250 1250
+Wire Wire Line
+	1250 1250 1250 1650
+Connection ~ 1250 1650
+Wire Wire Line
+	1250 1650 1350 1650
+Wire Wire Line
+	1350 1650 3000 1650
+Connection ~ 1350 1650
+Wire Wire Line
+	3350 2700 3750 2700
+$Comp
+L Connector:TestPoint_Probe TP1
+U 1 1 5F0D681E
+P 9650 6950
+F 0 "TP1" H 9803 7052 50  0000 L CNN
+F 1 "TestPoint_Probe" H 9803 6961 50  0000 L CNN
+F 2 "footprints:KB_BlueMicro" H 9850 6950 50  0001 C CNN
+F 3 "~" H 9850 6950 50  0001 C CNN
+	1    9650 6950
+	1    0    0    -1
+$EndComp
+$Comp
+L Mechanical:MountingHole MH1
+U 1 1 5F0D697D
+P 8700 6900
+F 0 "MH1" H 8800 6946 50  0000 L CNN
+F 1 "MountingHole" H 8800 6855 50  0000 L CNN
+F 2 "kbd:HOLE_JLCPCBA" H 8700 6900 50  0001 C CNN
+F 3 "~" H 8700 6900 50  0001 C CNN
+	1    8700 6900
+	1    0    0    -1
+$EndComp
+$Comp
+L Mechanical:MountingHole MH2
+U 1 1 5F0D6A17
+P 8700 7150
+F 0 "MH2" H 8800 7196 50  0000 L CNN
+F 1 "MountingHole" H 8800 7105 50  0000 L CNN
+F 2 "kbd:HOLE_JLCPCBA" H 8700 7150 50  0001 C CNN
+F 3 "~" H 8700 7150 50  0001 C CNN
+	1    8700 7150
+	1    0    0    -1
+$EndComp
 $EndSCHEMATC
