File: hardware/bmp/bmp.kicad_pcb (KiCad board)
At the start: 2 copper layers, 50.8 x 22.9 mm, 48 parts, among them J1 USB_C_Receptacle, J2 TC2050-IDC, J3 Conn_02x05_Odd_Even, J4 Conn_01x03, J5 Conn_01x04, Q1 SI2301CDS-T1-GE3, SW1 SW_Push, SW2 SW_Push, U1 XC6206P332MR, U2 STM32F103CBTx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

Commit message: updated with 2019 gdb
Parts:
- removed G***: LOGO, footprints:KB_BlueMicro
- removed R6: 10k, Resistor_SMD:R_0603_1608Metric
- removed Ref** (x2): Val**, kbd:HOLE_JLCPCBA
- removed SW1: SW_Push, footprints:SW_TACT_TS-1145A_C318904
- added MH1: MountingHole, kbd:HOLE_JLCPCBA, F.Cu at (68.6, 27.9)
- added MH2: MountingHole, kbd:HOLE_JLCPCBA, F.Cu at (27.3, 46.4)
- added TP1: TestPoint_Probe, footprints:KB_BlueMicro, B.Cu at (47.0, 38.6)
- U1: value XC6206P332MR -> AP2112K-3.3; footprint Package_TO_SOT_SMD:SOT-23 -> Package_TO_SOT_SMD:SOT-23-5
- U3: value LOGIC-TXS0108EPWR(TSSOP20) -> TXS0108EPWR
- moved R15 18.0 mm to (53.8, 46.4), turned to 0 degrees
- moved SW2 17.1 mm to (47.0, 45.7), turned to 180 degrees
- moved R16 14.4 mm to (56.4, 28.5), turned to 90 degrees
- moved C8 14.3 mm to (54.7, 28.5)
- moved J3 10.5 mm to (68.6, 40.6), turned to 180 degrees
- moved C5 8.89 mm to (53.1, 28.6)
- moved R14 8.64 mm to (51.4, 28.5)
- moved R13 8.13 mm to (49.8, 28.5)
- moved Q1 7.82 mm to (46.9, 28.2), turned to 0 degrees
- moved R17 6.09 mm to (57.6, 46.4), turned to 0 degrees
- moved R18 5.61 mm to (57.6, 44.5), turned to 0 degrees
- moved R20 5.21 mm to (60.1, 40.8)
- moved R21 5.21 mm to (58.4, 40.8)
- moved R19 5.21 mm to (61.7, 40.8)
- moved C2 4.19 mm to (43.9, 28.3), turned to 90 degrees
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Connections:
- U1 pad 1: GND -> +5V
- U1 pad 2: +3V3 -> GND
- U2 pad 44: Net-(R6-Pad1) -> GND
Routing:
- net GND: track 185.3 -> 146.6 mm, vias 24 -> 28
- net Net-(R6-Pad1): track 21.6 -> 0.00 mm, vias 2 -> 0
- net /TMS: track 31.5 -> 10.6 mm
- net /TPWR: track 53.6 -> 39.8 mm, vias 1 -> 0
- net Net-(C8-Pad1): track 11.6 -> 24.6 mm
- net /TCK: track 24.1 -> 15.6 mm
- net /BOOTLOADER: track 13.2 -> 21.0 mm, vias 0 -> 2
- net Net-(R17-Pad1): track 2.25 -> 9.15 mm
- net /RST: track 12.7 -> 18.9 mm, vias 0 -> 1
- net /TARGET_POWER_ADC: track 15.8 -> 10.1 mm
- net +3V3: track 94.7 -> 89.1 mm, vias 5 -> 3
- net Net-(R18-Pad1): track 2.39 -> 7.33 mm
- net /PWR_BB: track 11.1 -> 7.06 mm
- net Net-(J1-PadA5): track 8.13 -> 4.16 mm, vias 2 -> 0
- net /iRST: track 13.0 -> 16.8 mm, vias 2 -> 0
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Other:
- board size 50.8 x 22.9 mm -> 45.7 x 22.9 mm
- board text added: "2020-07-01"
- board text added: "CLK"
- board text added: "GND"
- board text added: "GND NC GND GND TPWR"
- board text added: "IO"
- board text added: "IO CLK GND TPWR"
- board text added: "RST TDI TDO TCK TMS"
- board text added: "SERIAL 3.3V"
- board text added: "SWD 1.8-3.3V"
- board text added: "SWO"
- board text added: "TPWR"
- board text added: "TPWR GND CLK IO"
- board text added: "TX RX GND"
- board text added: "github.com/jpconstantineau/NRF52-GDB-Debugger"
- board text added: "nRF52 GDB Debugger"
- board text removed: "Boot0"
- board text removed: "GND PWR"
- board text removed: "IO CLK GND PWR"
- board text removed: "SWO CLK IO"
- board text removed: "TMS TCK TDO TDI RST"
- board text removed: "TPWR GND GND NC GND"
- board text removed: "TPWR GND TCK TMS"
- board text removed: "TXD RXD GND"
- board text removed: "nRF52 GDB Debugger - 2020-06-15"

Commit message: update to the scripts
Other:
- board text added: "JLCJLCJLCJLC"
